File: YetAnotherKeyboard.kicad_sch (KiCad schematic)
At the start: 12 parts, among them SW88 SW_SPDT, U1 TP4056-42-ESOP8

Commit message: rev 1.1
Parts:
- added D88: Green LED, LED_SMD:LED_0603_1608Metric, symbol Device:LED
- added D89: Red LED, LED_SMD:LED_0603_1608Metric, symbol Device:LED
- added U2: ER_OLEDM0.91_1x-I2C, Display:ER_OLEDM0.91_1x-I2C, symbol Display_Graphic:ER_OLEDM0.91_1x-I2C
Connections:
- net GND: now also U2.1 (GND)
- net at R1.2, R2.1: now also A2.34 (GPIO28_ADC2); no longer A2.31 (GPIO26_ADC0)
- net at C2.1, R3.2, U1.4 (V_{CC})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: now also D88.1 (K), D89.1 (K)
- net +3V3: now reaches A2.36 (3V3)
- net +3V3: now also U2.2 (VCC)
- net CHRG: no longer names the net of U1.7 (~{CHRG})
- net CHRG: now also D89.2 (A); no longer A2.32 (GPIO27_ADC1)
- net STDBY: no longer names the net of U1.6 (~{STDBY})
- net STDBY: now also D88.2 (A); no longer A2.34 (GPIO28_ADC2)
- new net SCL: A2.32 (GPIO27_ADC1), U2.3 (SCL)
- new net SDA: A2.31 (GPIO26_ADC0), U2.4 (SDA)
- no-connect marks 5 -> 4
Other:
- note added: "A 128x64 1.54" oled will be used but there is no built-in KiCad footprint for that and this footprint is pin compatible LCSC part number:C7465999"
