File: matrix.kicad_sch (KiCad schematic)
At the start: 174 parts, among them SW1 ESC, SW10 F9, SW11 F10, SW12 F11, SW13 F12, SW14 PrSc, SW15 ScLk, SW16 Pause, SW17 `, SW18 1, SW19 2, SW2 F1, SW20 3, SW21 4, SW22 5, SW23 6, SW24 7, SW25 8, SW26 9, SW27 0, SW28 -, SW29 =, SW3 F2, SW30 Backspace, SW31 Ins, SW32 Home, SW33 PgUp, SW34 Tab, SW35 Q, SW36 W, SW37 E, SW38 R, SW39 T, SW4 F3, SW40 Y, SW41 U, SW42 I, SW43 O, SW44 P, SW45 [, SW46 ], SW47 \, SW48 Del, SW49 End, SW5 F4, SW50 PgDn, SW51 CapsLk, SW52 A, SW53 S, SW54 D, SW55 F, SW56 G, SW57 H, SW58 J, SW59 K, SW6 F5, SW60 L, SW61 ;, SW62 ', SW63 Enter, SW64 Shift, SW65 Z, SW66 X, SW67 C, SW68 V, SW69 B, SW7 F6, SW70 N, SW71 M, SW72 ,, SW73 ., SW74 /, SW75 Shift, SW76 Up, SW77 Ctrl, SW78 Win, SW79 Alt, SW8 F7, SW80 Space, SW81 Alt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

Commit message: rev 1.1
Parts:
- added D91, D92, D93, D94: 1N4148, Diode_SMD:D_SOD-123, symbol Device:D
- added SW89: M1, MX_Hotswap:MX-Hotswap-1U, symbol Switch:SW_Push
- added SW90: M2, MX_Hotswap:MX-Hotswap-1U, symbol Switch:SW_Push
- added SW91: M3, MX_Hotswap:MX-Hotswap-1U, symbol Switch:SW_Push
- added SW92: M4, MX_Hotswap:MX-Hotswap-1U, symbol Switch:SW_Push
Connections:
- net COL16: now also SW89.2, SW91.2
- net COL17: now also SW90.2, SW92.2
- net ROW5: now also D91.1 (K), D92.1 (K)
- net ROW6: now also D93.1 (K), D94.1 (K)
- new net: D91.2 (A), SW89.1
- new net: D92.2 (A), SW90.1
- new net: D93.2 (A), SW91.1
- new net: D94.2 (A), SW92.1
