File: YetAnotherKeyboard.kicad_pcb (KiCad board)
At the start: 2 copper layers, 422.3 x 138.1 mm, 186 parts, among them SW1 ESC, SW10 F9, SW11 F10, SW12 F11, SW13 F12, SW14 PrSc, SW15 ScLk, SW16 Pause, SW17 `, SW18 1, SW19 2, SW2 F1, SW20 3, SW21 4, SW22 5, SW23 6, SW24 7, SW25 8, SW26 9, SW27 0, SW28 -, SW29 =, SW3 F2, SW30 Backspace, SW31 Ins, SW32 Home, SW33 PgUp, SW34 Tab, SW35 Q, SW36 W, SW37 E, SW38 R, SW39 T, SW4 F3, SW40 Y, SW41 U, SW42 I, SW43 O, SW44 P, SW45 [, SW46 ], SW47 \, SW48 Del, SW49 End, SW5 F4, SW50 PgDn, SW51 CapsLk, SW52 A, SW53 S, SW54 D, SW55 F, SW56 G, SW57 H, SW58 J, SW59 K, SW6 F5, SW60 L, SW61 ;, SW62 ', SW63 Enter, SW64 Shift, SW65 Z, SW66 X, SW67 C, SW68 V, SW69 B, SW7 F6, SW70 N, SW71 M, SW72 ,, SW73 ., SW74 /, SW75 Shift, SW76 Up, SW77 Ctrl, SW78 Win, SW79 Alt, SW8 F7, SW80 Space, SW81 Alt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

Commit message: rev 1.1
Parts:
- added D88: Green LED, LED_SMD:LED_0603_1608Metric, F.Cu at (509.5, 159.5)
- added D89: Red LED, LED_SMD:LED_0603_1608Metric, F.Cu at (513.5, 159.5)
- added D91: 1N4148, Diode_SMD:D_SOD-123, F.Cu at (478.6, 273.8)
- added D92: 1N4148, Diode_SMD:D_SOD-123, F.Cu at (497.7, 273.8)
- added D93: 1N4148, Diode_SMD:D_SOD-123, F.Cu at (478.6, 292.9)
- added D94: 1N4148, Diode_SMD:D_SOD-123, F.Cu at (497.7, 292.9)
- added SW89: M1, MX_Hotswap:MX-Hotswap-1U, F.Cu at (470.1, 266.9)
- added SW90: M2, MX_Hotswap:MX-Hotswap-1U, F.Cu at (489.1, 266.9)
- added SW91: M3, MX_Hotswap:MX-Hotswap-1U, F.Cu at (470.1, 285.9)
- added SW92: M4, MX_Hotswap:MX-Hotswap-1U, F.Cu at (489.1, 285.9)
- added U2: ER_OLEDM0.91_1x-I2C, Display:ER_OLEDM0.91_1x-I2C, F.Cu at (475.6, 220.6)
- moved R2 12.4 mm to (505.7, 172.6)
- moved R1 5.62 mm to (509.2, 176.1), turned to 0 degrees
- moved TP2 5.61 mm to (513.5, 234.0)
- moved TP1 3.00 mm to (508.2, 234.2)
Connections:
- A2 pad 31: Net-(A2-GPIO26_ADC0) -> /SDA
- A2 pad 32: /CHRG -> /SCL
- A2 pad 34: /STDBY -> Net-(A2-GPIO28_ADC2)
- A2 pad 36: unconnected-(A2-3V3-Pad36) -> +3V3
- R1 pad 2: Net-(A2-GPIO26_ADC0) -> Net-(A2-GPIO28_ADC2)
- R2 pad 1: Net-(A2-GPIO26_ADC0) -> Net-(A2-GPIO28_ADC2)
- U1 pad 6: /STDBY -> Net-(D88-A)
- U1 pad 7: /CHRG -> Net-(D89-A)
Routing:
- net COL17: track 93.9 -> 206.8 mm, vias 3 -> 4
- net +3V3: track 0.00 -> 112.8 mm, vias 0 -> 2
- net /SCL: track 0.00 -> 101.6 mm, vias 0 -> 2
- net /SDA: track 0.00 -> 95.7 mm, vias 0 -> 2
- net COL16: track 123.7 -> 210.6 mm
- net Net-(D88-A): track 0.00 -> 82.3 mm, vias 0 -> 2
- net Net-(D89-A): track 0.00 -> 79.1 mm, vias 0 -> 2
- net Net-(D88-K): track 23.3 -> 102.2 mm, vias 0 -> 2
- net /STDBY: track 72.9 -> 0.00 mm, vias 2 -> 0
- net /CHRG: track 70.1 -> 0.00 mm, vias 2 -> 0
- net ROW6: track 478.5 -> 527.5 mm
- net ROW5: track 444.7 -> 466.2 mm
- net /BAT: track 101.2 -> 90.0 mm
- net Net-(A2-GPIO28_ADC2): track 0.00 -> 10.3 mm
- net Net-(A2-GPIO26_ADC0): track 9.50 -> 0.00 mm
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Other:
- board size 422.3 x 138.1 mm -> 414.8 x 138.1 mm
- board text added: "BT+"
- board text added: "BT-"
- board text removed: "Battery"

Commit message: silkscreens
Parts:
- added G***: LOGO, LOGO, B.Cu at (476.1, 182.3)
- added G***: LOGO, LOGO, B.Cu at (279.9, 181.0)
- added G***: LOGO, LOGO, B.Cu at (391.7, 202.1)
- added G***: LOGO, LOGO, B.Cu at (327.5, 266.2)
- added G***: LOGO, LOGO, B.Cu at (180.8, 223.8)
- added G***: LOGO, LOGO, B.Cu at (132.2, 176.1)
Other:
- board text added: "YetAnotherKeyboard rev 1.1"
- board text added: "github.com/0x62b/YetAnotherKeyboard"
- board text added: "github: @0x62b hc slack: @0x62 web: 0x62.dev"
- board text added: "soup!"
