File: PCB/YetAnotherKeyboard.kicad_pcb (KiCad board)
At the start: 2 copper layers, 414.8 x 138.1 mm, 203 parts, among them SW1 ESC, SW10 F9, SW11 F10, SW12 F11, SW13 F12, SW14 PrSc, SW15 ScLk, SW16 Pause, SW17 `, SW18 1, SW19 2, SW2 F1, SW20 3, SW21 4, SW22 5, SW23 6, SW24 7, SW25 8, SW26 9, SW27 0, SW28 -, SW29 =, SW3 F2, SW30 Backspace, SW31 Ins, SW32 Home, SW33 PgUp, SW34 Tab, SW35 Q, SW36 W, SW37 E, SW38 R, SW39 T, SW4 F3, SW40 Y, SW41 U, SW42 I, SW43 O, SW44 P, SW45 [, SW46 ], SW47 \, SW48 Del, SW49 End, SW5 F4, SW50 PgDn, SW51 CapsLk, SW52 A, SW53 S, SW54 D, SW55 F, SW56 G, SW57 H, SW58 J, SW59 K, SW6 F5, SW60 L, SW61 ;, SW62 ', SW63 Enter, SW64 Shift, SW65 Z, SW66 X, SW67 C, SW68 V, SW69 B, SW7 F6, SW70 N, SW71 M, SW72 ,, SW73 ., SW74 /, SW75 Shift, SW76 Up, SW77 Ctrl, SW78 Win, SW79 Alt, SW8 F7, SW80 Space, SW81 Alt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

Commit message: 65% pcb
Parts:
- removed A2: RaspberryPi_Pico_W, Module:RaspberryPi_Pico_W_SMD_HandSolder
- removed C1, C2: 10uF, Capacitor_SMD:C_0402_1005Metric
- removed D1, D67, D68, D69, D70, D71, D72, D73, D74, D75, D76, D77, D78, D79, D80, D81, D82, D83, D84, D85, D86, D87, D91, D92, D93, D94: 1N4148, Diode_SMD:D_SOD-123
- removed D88: Green LED, LED_SMD:LED_0603_1608Metric
- removed D89: Red LED, LED_SMD:LED_0603_1608Metric
- removed D90: 1N5819, Diode_THT:D_DO-41_SOD81_P7.62mm_Horizontal
- removed G*** (x6): LOGO, LOGO
- removed R2: 100kΩ, Resistor_SMD:R_0402_1005Metric
- removed R3: 0.4Ω, Resistor_SMD:R_0402_1005Metric
- removed R4: 2KΩ, Resistor_SMD:R_0402_1005Metric
- removed SW67: C, MX_Hotswap:MX-Hotswap-1U
- removed SW68: V, MX_Hotswap:MX-Hotswap-1U
- removed SW69: B, MX_Hotswap:MX-Hotswap-1U
- removed SW70: N, MX_Hotswap:MX-Hotswap-1U
- removed SW71: M, MX_Hotswap:MX-Hotswap-1U
- removed SW72: ,, MX_Hotswap:MX-Hotswap-1U
- removed SW73: ., MX_Hotswap:MX-Hotswap-1U
- removed SW74: /, MX_Hotswap:MX-Hotswap-1U
- removed SW75: Shift, MX_Hotswap:MX-Hotswap-2.75U
- removed SW76: Up, MX_Hotswap:MX-Hotswap-1U
- removed SW77, SW84: Ctrl, MX_Hotswap:MX-Hotswap-1.25U
- removed SW78, SW82: Win, MX_Hotswap:MX-Hotswap-1.25U
- removed SW79, SW81: Alt, MX_Hotswap:MX-Hotswap-1.25U
- removed SW80: Space, MX_Hotswap:MX-Hotswap-6.25U
- removed SW83: Menu, MX_Hotswap:MX-Hotswap-1.25U
- removed SW85: Left, MX_Hotswap:MX-Hotswap-1U
- removed SW86: Down, MX_Hotswap:MX-Hotswap-1U
- removed SW87: Right, MX_Hotswap:MX-Hotswap-1U
- removed SW88: SW_SPDT, Button_Switch_SMD:SW_SPDT_Shouhan_MSK12C02
- removed SW89: M1, MX_Hotswap:MX-Hotswap-1U
- removed SW90: M2, MX_Hotswap:MX-Hotswap-1U
- removed SW91: M3, MX_Hotswap:MX-Hotswap-1U
- removed SW92: M4, MX_Hotswap:MX-Hotswap-1U
- removed U2: ER_OLEDM0.91_1x-I2C, Display:ER_OLEDM0.91_1x-I2C
- added J1: Conn_01x05, Connector_PinHeader_1.27mm:PinHeader_1x05_P1.27mm_Horizontal, F.Cu at (373.9, 263.2)
- R1: value 100kΩ -> 1K
- SW1: value ESC -> SW_Push; footprint MX_Hotswap:MX-Hotswap-1U -> Button_Switch_SMD:SW_Push_SPST_NO_Alps_SKRK
- SW10: value F9 -> 8
- SW11: value F10 -> 9
- SW12: value F11 -> 0
- SW13: value F12 -> \; footprint MX_Hotswap:MX-Hotswap-1U -> MX_Hotswap:MX-Hotswap-1.5U
- SW14: value PrSc -> Backspace; footprint MX_Hotswap:MX-Hotswap-1U -> MX_Hotswap:MX-Hotswap-2U
- SW15: value ScLk -> Tab; footprint MX_Hotswap:MX-Hotswap-1U -> MX_Hotswap:MX-Hotswap-1.5U
- SW16: value Pause -> Q
- SW17: value ` -> W
- SW18: value 1 -> E
- SW19: value 2 -> R
- SW2: value F1 -> ESC
- SW20: value 3 -> T
- SW21: value 4 -> Y
- SW22: value 5 -> U
- SW23: value 6 -> I
- SW24: value 7 -> O
- SW25: value 8 -> P
- SW26: value 9 -> -
- SW27: value 0 -> =
- SW28: value - -> CapsLk; footprint MX_Hotswap:MX-Hotswap-1U -> MX_Hotswap:MX-Hotswap-1.75U
- SW29: value = -> A
- SW3: value F2 -> 1
- SW30: value Backspace -> S; footprint MX_Hotswap:MX-Hotswap-2U -> MX_Hotswap:MX-Hotswap-1U
- SW31: value Ins -> D
- SW32: value Home -> F
- SW33: value PgUp -> G
- SW34: value Tab -> H; footprint MX_Hotswap:MX-Hotswap-1.5U -> MX_Hotswap:MX-Hotswap-1U
- SW35: value Q -> J
- SW36: value W -> K
- SW37: value E -> L
- SW38: value R -> ;
- SW39: value T -> [
- SW4: value F3 -> 2
- SW40: value Y -> ]
- SW41: value U -> Shift; footprint MX_Hotswap:MX-Hotswap-1U -> MX_Hotswap:MX-Hotswap-2.25U
- SW42: value I -> Z
- SW43: value O -> X
- SW44: value P -> C
- SW45: value [ -> V
- SW46: value ] -> B
- SW47: value \ -> N; footprint MX_Hotswap:MX-Hotswap-1.5U -> MX_Hotswap:MX-Hotswap-1U
- SW48: value Del -> M
- SW49: value End -> ,
- SW5: value F4 -> 3
- SW50: value PgDn -> .
- SW51: value CapsLk -> /; footprint MX_Hotswap:MX-Hotswap-1.75U -> MX_Hotswap:MX-Hotswap-1U
- SW52: value A -> '
- SW53: value S -> Enter; footprint MX_Hotswap:MX-Hotswap-1U -> MX_Hotswap:MX-Hotswap-2.25U
- SW54: value D -> Ctrl; footprint MX_Hotswap:MX-Hotswap-1U -> MX_Hotswap:MX-Hotswap-1.25U
- SW55: value F -> Win; footprint MX_Hotswap:MX-Hotswap-1U -> MX_Hotswap:MX-Hotswap-1.25U
- SW56: value G -> Alt; footprint MX_Hotswap:MX-Hotswap-1U -> MX_Hotswap:MX-Hotswap-1.25U
- SW57: value H -> Space; footprint MX_Hotswap:MX-Hotswap-1U -> MX_Hotswap:MX-Hotswap-6.25U
- SW58: value J -> Alt; footprint MX_Hotswap:MX-Hotswap-1U -> MX_Hotswap:MX-Hotswap-1.25U
- SW59: value K -> Fn; footprint MX_Hotswap:MX-Hotswap-1U -> MX_Hotswap:MX-Hotswap-1.25U
- SW6: value F5 -> 4
- SW60: value L -> Left
- SW61: value ; -> Down
- SW62: value ' -> Right
- SW63: value Enter -> Shift; footprint MX_Hotswap:MX-Hotswap-2.25U -> MX_Hotswap:MX-Hotswap-1.75U
- SW64: value Shift -> Up; footprint MX_Hotswap:MX-Hotswap-2.25U -> MX_Hotswap:MX-Hotswap-1U
- SW65: value Z -> Del
- SW66: value X -> Ins
- SW7: value F6 -> 5
- SW8: value F7 -> 6
- SW9: value F8 -> 7
- TP1: value BT+ -> BAT; footprint TestPoint:TestPoint_Pad_D4.0mm -> TestPoint:TestPoint_Pad_D2.0mm
- TP2: value BT- -> GND; footprint TestPoint:TestPoint_Pad_D4.0mm -> TestPoint:TestPoint_Pad_D2.0mm
- U1: value TP4056-42-ESOP8 -> nice_nano; footprint Package_SO:SOIC-8-1EP_3.9x4.9mm_P1.27mm_EP2.41x3.3mm_ThermalVias -> nice_nano:nice_nano
- moved SW15 344.4 mm to (87.5, 236.7)
- moved D16 342.0 mm to (117.5, 244.5), turned to 0 degrees
- moved D15 342.0 mm to (98.5, 244.5), turned to 0 degrees
- moved SW16 339.7 mm to (111.3, 236.7)
- moved SW1 287.4 mm to (393.2, 245.3)
- moved D32 260.7 mm to (179.3, 263.5), turned to 0 degrees
- moved D33 260.7 mm to (198.4, 263.5), turned to 0 degrees
- moved D31 260.6 mm to (160.3, 263.5), turned to 0 degrees
- moved SW33 258.3 mm to (192.2, 255.7)
- moved SW31 258.3 mm to (154.1, 255.7)
- moved SW32 258.3 mm to (173.2, 255.7)
- moved D30 251.2 mm to (141.3, 263.5), turned to 0 degrees
- moved SW30 239.6 mm to (135.1, 255.7)
- moved SW28 237.2 mm to (89.9, 255.7)
- moved D28 232.6 mm to (103.2, 263.5), turned to 0 degrees
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Connections:
- D15 pad 1: ROW1 -> ROW2
- D16 pad 1: ROW1 -> ROW2
- D28 pad 1: ROW2 -> ROW3
- D29 pad 1: ROW2 -> ROW3
- D30 pad 1: ROW2 -> ROW3
- D31 pad 1: ROW2 -> ROW3
- D32 pad 1: ROW2 -> ROW3
- D33 pad 1: ROW2 -> ROW3
- D41 pad 1: ROW3 -> ROW4
- D42 pad 1: ROW3 -> ROW4
- D43 pad 1: ROW3 -> ROW4
- D44 pad 1: ROW3 -> ROW4
- D45 pad 1: ROW3 -> ROW4
- D46 pad 1: ROW3 -> ROW4
- D47 pad 1: ROW3 -> ROW4
- D48 pad 1: ROW3 -> ROW4
- D49 pad 1: ROW3 -> ROW4
- D50 pad 1: ROW3 -> ROW4
- D54 pad 1: ROW4 -> ROW5
- D55 pad 1: ROW4 -> ROW5
- D56 pad 1: ROW4 -> ROW5
- D57 pad 1: ROW4 -> ROW5
- D58 pad 1: ROW4 -> ROW5
- D59 pad 1: ROW4 -> ROW5
- D60 pad 1: ROW4 -> ROW5
- D61 pad 1: ROW4 -> ROW5
- D62 pad 1: ROW4 -> ROW5
- D63 pad 1: ROW4 -> ROW5
- R1 pad 1: /BAT -> Net-(U1-RST)
- R1 pad 2: Net-(A2-GPIO28_ADC2) -> Net-(R1-Pad2)
- SW1 pad 1: Net-(D1-A) -> Net-(R1-Pad2)
- SW1 pad 2: COL1 -> GND
- SW10 pad 2: COL10 -> COL9
- SW11 pad 2: COL11 -> COL10
- SW12 pad 2: COL12 -> COL11
- SW13 pad 2: COL13 -> COL12
- SW14 pad 2: COL14 -> COL13
- SW15 pad 2: COL15 -> COL1
- SW16 pad 2: COL16 -> COL2
- SW17 pad 2: COL1 -> COL3
- SW18 pad 2: COL2 -> COL4
- SW19 pad 2: COL3 -> COL5
- SW2 pad 2: COL2 -> COL1
- SW20 pad 2: COL4 -> COL6
- SW21 pad 2: COL5 -> COL7
- SW22 pad 2: COL6 -> COL8
- SW23 pad 2: COL7 -> COL9
- SW24 pad 2: COL8 -> COL10
- SW25 pad 2: COL9 -> COL11
- SW26 pad 2: COL10 -> COL12
- SW27 pad 2: COL11 -> COL13
- SW28 pad 2: COL12 -> COL1
- SW29 pad 2: COL13 -> COL2
- SW3 pad 2: COL3 -> COL2
- SW30 pad 2: COL14 -> COL3
- SW31 pad 2: COL15 -> COL4
- SW32 pad 2: COL16 -> COL5
- SW33 pad 2: COL17 -> COL6
- SW34 pad 2: COL1 -> COL7
- SW35 pad 2: COL2 -> COL8
- SW36 pad 2: COL3 -> COL9
- SW37 pad 2: COL4 -> COL10
- SW38 pad 2: COL5 -> COL11
- SW39 pad 2: COL6 -> COL12
- SW4 pad 2: COL4 -> COL3
- SW40 pad 2: COL7 -> COL13
- SW41 pad 2: COL8 -> COL1
- SW42 pad 2: COL9 -> COL2
- SW43 pad 2: COL10 -> COL3
- SW44 pad 2: COL11 -> COL4
- SW45 pad 2: COL12 -> COL5
- SW46 pad 2: COL13 -> COL6
- SW47 pad 2: COL14 -> COL7
- SW48 pad 2: COL15 -> COL8
- SW49 pad 2: COL16 -> COL9
- SW5 pad 2: COL5 -> COL4
- SW50 pad 2: COL17 -> COL10
- SW51 pad 2: COL1 -> COL11
- SW52 pad 2: COL2 -> COL12
- SW53 pad 2: COL3 -> COL13
- SW54 pad 2: COL4 -> COL1
- SW55 pad 2: COL5 -> COL2
- SW56 pad 2: COL6 -> COL3
- SW57 pad 2: COL7 -> COL4
- SW58 pad 2: COL8 -> COL5
- SW59 pad 2: COL9 -> COL6
- SW6 pad 2: COL6 -> COL5
- SW60 pad 2: COL10 -> COL7
- SW61 pad 2: COL11 -> COL8
- SW62 pad 2: COL12 -> COL9
- SW63 pad 2: COL13 -> COL10
- SW64 pad 2: COL1 -> COL11
- SW65 pad 2: COL2 -> COL12
- SW66 pad 2: COL3 -> COL13
- SW7 pad 2: COL7 -> COL6
- SW8 pad 2: COL8 -> COL7
- SW9 pad 2: COL9 -> COL8
- TP1 pad 1: /BAT -> Net-(U1-BATIN/P0.04)
- U1 pad 1: GND -> /CS
- U1 pad 2: Net-(U1-PROG) -> COL1
- U1 pad 4: Net-(D88-K) -> GND
- U1 pad 5: /BAT -> /MOSI
- U1 pad 6: Net-(D88-A) -> /SCK
- U1 pad 7: Net-(D89-A) -> COL2
- U1 pad 8: Net-(D88-K) -> COL3
- U1 pad 9: GND -> COL4
Routing:
- net ROW6: track 527.5 -> 0.00 mm, vias 2 -> 0
- net COL10: track 448.5 -> 231.5 mm, vias 6 -> 5
- net COL16: track 210.6 -> 0.00 mm, vias 3 -> 0
- net COL11: track 426.5 -> 217.1 mm, vias 6 -> 8
- net COL17: track 206.8 -> 0.00 mm, vias 4 -> 0
- net COL9: track 464.6 -> 265.1 mm
- net COL6: track 498.8 -> 301.6 mm
- net COL5: track 521.9 -> 334.8 mm
- net COL8: track 468.0 -> 285.2 mm, vias 6 -> 10
- net COL7: track 483.2 -> 302.6 mm, vias 6 -> 5
- net COL14: track 174.6 -> 0.00 mm, vias 3 -> 0
- net COL15: track 140.4 -> 0.00 mm, vias 3 -> 0
- net COL13: track 305.8 -> 171.5 mm, vias 5 -> 8
- net COL4: track 480.5 -> 364.9 mm, vias 6 -> 5
- net +3V3: track 112.8 -> 0.00 mm, vias 2 -> 0
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Other:
- board size 414.8 x 138.1 mm -> 329.7 x 98.2 mm
- board text added: "Battery"
- board text added: "HC Slack: @0x62 GitHub: @0x62b Website: https://0x62.dev Email: benjamin@0x62.dev"
- board text added: "YetAnotherKeyboard v2 https://github.com/0x62b/YetAnotherKeyboard"
- board text removed: "BT+"
- board text removed: "BT-"
- board text removed: "YetAnotherKeyboard rev 1.1"
- board text removed: "github.com/0x62b/YetAnotherKeyboard"
- board text removed: "github: @0x62b hc slack: @0x62 web: 0x62.dev"
- board text removed: "soup!"
