File: PCB/YetAnotherKeyboard.kicad_pcb (KiCad board)
At the start: 2 copper layers, 329.7 x 98.2 mm, 136 parts, among them J1 Conn_01x05, SW1 SW_Push, SW10 8, SW11 9, SW12 0, SW13 \, SW14 Backspace, SW15 Tab, SW16 Q, SW17 W, SW18 E, SW19 R, SW2 ESC, SW20 T, SW21 Y, SW22 U, SW23 I, SW24 O, SW25 P, SW26 -, SW27 =, SW28 CapsLk, SW29 A, SW3 1, SW30 S, SW31 D, SW32 F, SW33 G, SW34 H, SW35 J, SW36 K, SW37 L, SW38 ;, SW39 [, SW4 2, SW40 ], SW41 Shift, SW42 Z, SW43 X, SW44 C, SW45 V, SW46 B, SW47 N, SW48 M, SW49 ,, SW5 3, SW50 ., SW51 /, SW52 ', SW53 Enter, SW54 Ctrl, SW55 Win, SW56 Alt, SW57 Space, SW58 Alt, SW59 Fn, SW6 4, SW60 Left, SW61 Down, SW62 Right, SW63 Shift, SW64 Up, SW65 Del, SW66 Ins, SW7 5, SW8 6, SW9 7, U1 nice_nano

Commit message: idk
Parts:
- D10, D11, D12, D13, D14, D15, D16, D17, D18, D19, D2, D20, D21, D22, D23, D24, D25, D26, D27, D28, D29, D3, D30, D31, D32, D33, D34, D35, D36, D37, D38, D39, D4, D40, D41, D42, D43, D44, D45, D46, D47, D48, D49, D5, D50, D51, D52, D53, D54, D55, D56, D57, D58, D59, D6, D60, D61, D62, D63, D64, D65, D66, D7, D8, D9, SW10, SW11, SW12, SW13, SW14, SW15, SW16, SW17, SW18, SW19, SW2, SW20, SW21, SW22, SW23, SW24, SW25, SW26, SW27, SW28, SW29, SW3, SW30, SW31, SW32, SW33, SW34, SW35, SW36, SW37, SW38, SW39, SW4, SW40, SW41, SW42, SW43, SW44, SW45, SW46, SW47, SW48, SW49, SW5, SW50, SW51, SW52, SW53, SW54, SW55, SW56, SW57, SW58, SW59, SW6, SW60, SW61, SW62, SW63, SW64, SW65, SW66, SW7, SW8, SW9: moved to B.Cu
- moved D57 112.4 mm to (148.0, 301.6), turned to 180 degrees
- moved D41 36.2 mm to (76.5, 282.6), turned to 180 degrees
- moved D53 36.1 mm to (319.4, 263.5), turned to 180 degrees
- moved D14 32.6 mm to (323.8, 225.4), turned to 180 degrees
- moved D63 26.7 mm to (309.9, 282.6), turned to 180 degrees
- moved D28 26.7 mm to (76.5, 263.5), turned to 180 degrees
- moved D15 22.0 mm to (76.5, 244.5), turned to 180 degrees
- moved D13 21.8 mm to (333.8, 244.5), turned to 180 degrees
- moved D58 17.2 mm to (266.9, 301.6), turned to 180 degrees
- moved D59 17.1 mm to (290.8, 301.6), turned to 180 degrees
- moved D55 17.1 mm to (100.3, 301.6), turned to 180 degrees
- moved D54 17.1 mm to (76.5, 301.6), turned to 180 degrees
- moved D56 17.0 mm to (124.2, 301.6), turned to 180 degrees
- moved D44 12.6 mm to (157.3, 282.6), turned to 180 degrees
- moved D46 12.6 mm to (195.4, 282.6), turned to 180 degrees
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Routing:
- net COL1: track 508.0 -> 390.3 mm, vias 0 -> 5
- net COL12: track 265.0 -> 170.0 mm, vias 6 -> 9
- net COL2: track 475.7 -> 387.4 mm
- net COL3: track 437.8 -> 349.5 mm, vias 5 -> 6
- net GND: track 68.6 -> 9.51 mm, vias 6 -> 11
- net ROW4: track 328.6 -> 373.5 mm
- net COL10: track 231.5 -> 196.5 mm
- net COL7: track 302.6 -> 268.0 mm, vias 5 -> 6
- net COL5: track 334.8 -> 300.6 mm, vias 6 -> 8
- net COL11: track 217.1 -> 184.2 mm, vias 8 -> 9
- net /CS: track 55.1 -> 87.2 mm
- net ROW1: track 345.7 -> 375.6 mm, vias 2 -> 0
- net COL8: track 285.2 -> 260.0 mm, vias 10 -> 5
- net ROW3: track 328.6 -> 348.0 mm, vias 2 -> 1
- net COL13: track 171.5 -> 153.1 mm, vias 8 -> 6
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
Commit message: 3d models
Parts:
- J1: footprint Connector_PinHeader_1.27mm:PinHeader_1x05_P1.27mm_Horizontal -> Connector_PinHeader_2.54mm:PinHeader_1x05_P2.54mm_Vertical
- moved J1 9.38 mm to (364.5, 262.5)
- moved D14 0.33 mm to (323.4, 225.4)
Routing:
- net /SCK: track 57.6 -> 71.5 mm
- net /MOSI: track 61.4 -> 75.0 mm
- net /VCC: track 64.1 -> 73.4 mm
- net /CS: track 87.2 -> 92.8 mm
- net COL4: track 353.1 -> 354.9 mm
- net COL2: track 387.4 -> 388.5 mm
- net COL11: track 184.2 -> 185.2 mm
- net COL9: track 253.4 -> 254.4 mm
- net GND: track 9.51 -> 8.70 mm, vias 11 -> 12
